File: epi_ESP32 (2023_01_16 13_30_41 UTC).kicad_pcb (KiCad board)
At the start: 4 copper layers, 12.7 x 22.3 mm, 37 parts, among them J1 Conn_01x08, J2 Conn_01x08, J3 USB_C_Receptacle_USB2.0, SW1 SW_MEC_5G, SW2 SW_MEC_5G, U1 ESP32-C3, U2 RT9080, Y1 Crystal_GND24

Commit message: new revision
Parts:
- removed R1: 10kΩ, Resistor_SMD:R_0402_1005Metric
- J2: value Conn_01x08 -> Conn_01x09; footprint Connector_PinHeader_1.27mm:PinHeader_1x08_P1.27mm_Vertical -> Connector_PinSocket_1.27mm:PinSocket_1x09_P1.27mm_Vertical
- Y1: value Crystal_GND24 -> Crystal
Connections:
- J2 pad 6: IO8 -> IO10
- J2 pad 7: IO7 -> IO8
- J2 pad 8: IO6 -> IO7
- U1 pad 16: Net-(U1-GPIO10) -> IO10
Routing:
- net IO10: track 0.00 -> 3.53 mm, vias 0 -> 1
- net Net-(U1-GPIO10): track 1.61 -> 0.00 mm
- net IO6: track 5.69 -> 6.26 mm
- net IO8: track 5.58 -> 6.10 mm
- net IO7: track 5.57 -> 6.09 mm
Other:
- board size 12.7 x 22.3 mm -> 22.5 x 27.1 mm
- board text added: "10"
- board text added: "v1,2,2"
- board text removed: "v1,2,1"

Commit message: new gerbers
Other:
- board size 22.5 x 27.1 mm -> 12.7 x 22.3 mm
Changed lines of the file:
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@@
+	)
+	(gr_line
+		(start 93 55.4)
+		(end 98 55.4)
+		(stroke
+			(width 0.05588)
+			(type default)
+		)
+		(layer "Dwgs.User")
+	)
+	(gr_line
+		(start 110.5 55.4)
+		(end 115.5 55.4)
+		(stroke
+			(width 0.05588)
+			(type default)
+		)
+		(layer "Dwgs.User")
+	)
+	(gr_line
+		(start 99.6 77)
+		(end 99.6 72)
+		(stroke
+			(width 0.05588)
+			(type default)
+		)
+		(layer "Dwgs.User")
 	)
 	(gr_line
@@
 		(layer "Edge.Cuts")
 	)
-	(gr_line
-		(start 93 55.4)
-		(end 98 55.4)
-		(stroke
-			(width 0.05588)
-			(type default)
-		)
-		(layer "Edge.Cuts")
-	)
 	(gr_arc
 		(start 97.89 52.15)
@@
 	)
 	(gr_line
-		(start 110.5 55.4)
-		(end 115.5 55.4)
-		(stroke
-			(width 0.05588)
-			(type default)
-		)
-		(layer "Edge.Cuts")
-	)
-	(gr_line
 		(start 97.89 49.9185)
 		(end 99.668345 49.915247)
@@
 		)
 		(layer "Edge.Cuts")
-	)
-	(gr_line
-		(start 99.6 77)
-		(end 99.6 72)
-		(stroke
-			(width 0.05588)
-			(type default)
-		)
-		(layer "Edge.Cuts")
